File: hardware/pcb/master_slave/master_slave_carrier.kicad_sch (KiCad schematic)
At the start: 0 parts

Commit message: Update master_slave_carrier.kicad_sch
Parts:
- added F1: Polyfuse, symbol Device:Polyfuse
- added J1A: Master_A_Row, symbol Connector:Conn_01x19
- added J1B: Master_B_Row, symbol Connector:Conn_01x19
- added J2A: Slave_A_Row, symbol Connector:Conn_01x19
- added J2B: Slave_B_Row, symbol Connector:Conn_01x19
- added J3: USB_C_Power_In, symbol Connector:USB_C_Receptacle_USB2.0
- added J4A: PHASE_A_OUT, symbol Connector:Conn_01x02
- added J4B: PHASE_B_OUT, symbol Connector:Conn_01x02
- added J4C: PHASE_C_OUT, symbol Connector:Conn_01x02
- added J6: OLED_I2C_Header, symbol Connector:Conn_01x04
- added R4, R5: 4.7k (opt), symbol Device:R
- added RCC1, RCC2: 5.1k, symbol Device:R
- added SW1: Master_EN, symbol Switch:SW_Push
- added SW2: Slave_EN, symbol Switch:SW_Push
Other:
- note added: "5V_IN: J3-VBUS -> F1 -> J1A-19, J2A-19"
- note added: "CC pull-downs: J3-CC1->RCC1->GND, J3-CC2->RCC2->GND"
- note added: "EN switches (optional): SW1->J1A-2, SW2->J2A-2"
- note added: "GND: J3-GND -> J1B-1 -> J2B-1 -> J4A-2/J4B-2/J4C-2 -> J6-2"
- note added: "NET MAP (first-pass):"
- note added: "OLED: J1A-1(3V3)->J6-1, J1B-3(IO22)->J6-3, J1B-6(IO21)->J6-4"
- note added: "PHASE_A: J1A-9(IO25)->J4A-1 PHASE_B: J2A-9(IO25)->J4B-1 PHASE_C: J2A-10(IO26)->J4C-1"
- note added: "Pull-ups (optional): R4 SCL->3V3, R5 SDA->3V3"
- note added: "UART_RX_S2M: J2B-11(IO17) -> J1B-12(IO16)"
- note added: "UART_TX_M2S: J1B-11(IO17) -> J2B-12(IO16)"
